Commit message: 修改

File: urdf/chassis.xacro (robot description, xacro)
@@ -1,8 +1,7 @@
-<!-- 机器人的底盘 -->
 <?xml version="1.0"?>
 <robot xmlns:xacro="http://www.ros.org/wiki/xacro">
     <xacro:include filename="$(find my_robot)/urdf/common_inertial.xacro"/>
     <xacro:macro name="chassis" params="prefix">
-        <link name="{prefix}_base_link">
+        <link name="${prefix}_base_link">
             <!-- 视觉 -->
             <visual>
@@ -11,5 +10,5 @@
                     <box size="0.4 0.3 0.1"/>
                 </geometry>
-                <material name="darkgray"/>
+                <material name="dark_grey"/>
             </visual>
             <!-- 碰撞属性 -->

File: urdf/common_inertial.xacro (robot description, xacro)
@@ -1,3 +1,2 @@
-<!-- 这是一个通用的惯性和质量宏定义 -->
 <?xml version="1.0"?>
 <robot xmlns:xacro="http://www.ros.org/wiki/xacro">

File: urdf/my_robot.xacro (robot description, xacro)
@@ -1,4 +1,6 @@
 <?xml version="1.0"?>
 <robot xmlns:xacro="http://www.ros.org/wiki/xacro" name="my_robot">
+    <!-- 机器人命名空间前缀 -->
+    <xacro:property name="prefix" value="robot"/>
     <xacro:include filename="$(find my_robot)/urdf/materials.xacro"/>
     <xacro:include filename="$(find my_robot)/urdf/common_inertial.xacro"/>
@@ -6,12 +8,10 @@
     <xacro:include filename="$(find my_robot)/urdf/wheels.xacro"/>
     <xacro:include filename="$(find my_robot)/urdf/sensors.xacro"/>
-    <!-- 机器人命名空间前缀 -->
-    <xacro:property name="prefix" value="robot"/>
     <!-- 实例化部件 -->
     <xacro:chassis prefix="${prefix}"/>
     <xacro:wheel prefix="${prefix}" side="left"/>
     <xacro:wheel prefix="${prefix}" side="right"/>
-    <xacro:lidar prefix="${prefix}"/>
-    <xacro:camera prefix="${prefix}"/>
+    <!-- <xacro:lidar prefix="${prefix}"/>
+    <xacro:camera prefix="${prefix}"/> -->
     <!-- Gazebo 差速驱动插件 -->
     <gazebo>
@@ -23,6 +23,6 @@
             </ros>
             <update_rate>30.0</update_rate>
-            <left_wheel>${prefix}_left_wheel_joint</left_wheel>
-            <right_wheel>${prefix}_right_wheel_joint</right_wheel>
+            <left_joint>${prefix}_left_wheel_joint</left_joint>
+            <right_joint>${prefix}_right_wheel_joint</right_joint>
             <wheel_separation>0.4</wheel_separation>
             <wheel_diameter>0.1</wheel_diameter>
@@ -33,5 +33,5 @@
             <!-- 输出 -->
             <publish_odom>true</publish_odom>
-            <puplish_odom_tf>true</puplish_odom_tf>
+            <publish_odom_tf>true</publish_odom_tf>
             <publish_wheel_tf>true</publish_wheel_tf>
             <odometry_frame>odom</odometry_frame>
@@ -39,78 +39,3 @@
         </plugin>
     </gazebo>
-    <!-- Gazebo 激光雷达插件（使用 GPU 加速） -->
-    <gazebo reference="${prefix}_lidar_link">
-      <sensor name="lidar" type="gpu_ray">  <!-- 若需 CPU，改为 type="ray" -->
-        <pose>0 0 0 0 0 0</pose>
-        <topic>/points</topic>
-        <update_rate>10</update_rate>
-        <ray>
-          <scan>
-            <horizontal>
-              <samples>360</samples>
-              <resolution>1</resolution>
-              <min_angle>-3.14159</min_angle>
-              <max_angle>3.14159</max_angle>
-            </horizontal>
-            <vertical>
-              <samples>16</samples>
-              <min_angle>-0.261799</min_angle>  <!-- -15° -->
-              <max_angle>0.261799</max_angle>    <!-- 15° -->
-            </vertical>
-          </scan>
-          <range>
-            <min>0.5</min>
-            <max>30.0</max>
-            <resolution>0.01</resolution>
-          </range>
-          <noise>
-            <type>gaussian</type>
-            <mean>0.0</mean>
-            <stddev>0.01</stddev>
-          </noise>
-        </ray>
-        <plugin name="gazebo_ros_ray_sensor" filename="libgazebo_ros_ray_sensor.so">
-          <ros>
-            <namespace>/</namespace>
-            <remapping>~/points:=points</remapping>  <!-- 使用重映射 -->
-          </ros>
-          <output_type>sensor_msgs/PointCloud2</output_type>
-          <frame_name>${prefix}_lidar_link</frame_name>
-        </plugin>
-      </sensor>
-    </gazebo>
-     <!-- Gazebo 相机插件 -->
-    <gazebo reference="${prefix}_camera_link">
-      <sensor name="camera" type="camera">
-        <pose>0 0 0 0 0 0</pose>
-        <topic>/camera/image_raw</topic>
-        <update_rate>30</update_rate>
-        <camera>
-          <horizontal_fov>1.0472</horizontal_fov> <!-- 60° -->
-          <image>
-            <width>640</width>
-            <height>480</height>
-            <format>R8G8B8</format>
-          </image>
-          <clip>
-            <near>0.1</near>
-            <far>100</far>
-          </clip>
-          <noise>
-            <type>gaussian</type>
-            <mean>0.0</mean>
-            <stddev>0.01</stddev>
-          </noise>
-        </camera>
-        <plugin name="gazebo_ros_camera" filename="libgazebo_ros_camera.so">
-          <ros>
-            <namespace>/</namespace>
-            <remapping>~/image_raw:=camera/image_raw</remapping>
-            <remapping>~/camera_info:=camera/camera_info</remapping>
-          </ros>
-          <camera_name>camera</camera_name>
-          <frame_name>${prefix}_camera_link</frame_name>
-        </plugin>
-      </sensor>
-    </gazebo>
 </robot>

File: urdf/sensors.xacro (robot description, xacro)
@@ -21,7 +21,7 @@
             <xacro:cylinder_inertial m="0.1" r="0.05" h="0.1"/>
         </link>
-        <joint name="{prefix_lidar_joint}" type="fixed">
-            <parent link="{prefix}_base_link"/>
-            <child link="{prefix}_lidar_link"/>
+        <joint name="${prefix}_lidar_joint" type="fixed">
+            <parent link="${prefix}_base_link"/>
+            <child link="${prefix}_lidar_link"/>
             <!-- 安装位置：底盘前方中心（0.2-r），离地0.15（雷达底面离地0.15） -->
             <!-- 父坐标系：底盘底盘的几何中心，虽然抬高了0.05，但是坐标系原点不变 -->

File: urdf/wheels.xacro (robot description, xacro)
@@ -1,7 +1,15 @@
-<!-- 机器人的左右轮子 -->
 <?xml version="1.0"?>
 <robot xmlns:xacro="http://www.ros.org/wiki/xacro">
     <xacro:include filename="$(find my_robot)/urdf/common_inertial.xacro"/>
     <xacro:macro name="wheel" params="prefix side">
+        <!-- 根据 side 设置 y 偏移量 -->
+        <!-- <xacro:property name="y_offset" value="-0.2" if="side == 'left'"/>
+        <xacro:property name="y_offset" value="0.2" unless="side == 'left'"/> -->
+        <xacro:if value="${side == 'left'}">
+            <xacro:property name="y_offset" value="-0.2"/>
+        </xacro:if>
+        <xacro:unless value="${side == 'left'}">
+            <xacro:property name="y_offset" value="0.2"/>
+        </xacro:unless>
         <link name="${prefix}_${side}_wheel">
             <!-- 视觉 -->
@@ -11,5 +19,5 @@
                     <cylinder radius="0.05" length="0.05"/>
                 </geometry>
-                <material name="black">
+                <material name="black" />
             </visual>
             <!-- 碰撞 -->
@@ -28,7 +36,16 @@
             <child link="${prefix}_${side}_wheel"/>
             <!-- 轮子中心位置：x = -0.15（靠近后部），y 根据左右调整（0.3 / 2 + 0.05，使车轮在外部），z = 0.05（使轮子接地） -->
-            <origin xyz="-0.15 ${side == 'left' ? -0.2 : 0.2} 0.05" rpy="0 0 0"/>
+            <origin xyz="-0.15 ${y_offset} 0.051" rpy="0 0 0"/>
             <axis xyz="0 1 0"/> <!-- 绕 y 轴旋转 -->
         </joint>
+        <!-- 增加摩擦系数 -->
+        <gazebo reference="${prefix}_${side}_wheel">
+            <!-- <mu1 value="20.0" />
+            <mu2 value="20.0" />
+            <kp value="1000000000" />
+            <kd value="1.0" /> -->
+            <mu1>1.0</mu1>
+            <mu2>1.0</mu2>
+        </gazebo>
     </xacro:macro>
 </robot>
